File: haccess.sch (EAGLE design)
At the start: 1 part

Commit message: Think I'm done?
Parts:
- removed U$2: USB_RECESSED_C42620, pinebook_parts:USB_RECESSED_C42620
- added D1: (no value), SparkFun-LED:LED0603
- added R1: 160, rcl:R-EU_R0603
- added SAO: FEMALE 2x3, SparkFun-Connectors:CONN_03X2FEMALE
Connections:
- removed net 32U4_OSC: U$2.OUT
- removed net 5V: U$2.VBUS
- removed net DM4: U$2.D-
- removed net DP4: U$2.D+
- new net 3.3V: SAO.1
- new net D+: R1.2
- new net D_P: R1.1
- new net ISET: R1.1
- new net MIC: R1.1
- new net N$1: D1.A, R1.1
- new net SAO1: SAO.5
- new net SAO2: SAO.6
- new net SCL: SAO.4
- new net SDA: SAO.3
- new net SENSE: R1.1
- new net STATUS: R1.2
- net GND: now also D1.C, R1.2, SAO.2; no longer U$2.GND
- net VCC: now also R1.2; no longer U$2.EN, U$2.VCC

Commit message: I think I'm done?
Other:
- moved on the sheet: SAO

Commit message: More revisioning.. Now has always-available power.. but its not completed. Daughterboard dimensions completed.
Parts:
- added D2: (no value), SparkFun-LED:LED0603
- added R2: 160, rcl:R-EU_R0603
Connections:
- new net 5V: R2.1
- new net AUD_STATUS: R2.2
- new net D-: R2.2
- new net D_N: R2.1
- new net EN: R2.2
- new net GND_ISOLATED: SAO.2
- new net N$2: D2.A, R2.1
- net GND: now also D2.C; no longer SAO.2
